Commit message: .

File: src/rc_description/urdf/rc_base.urdf (robot description, URDF)
Before this commit: robot rc_car, 2 links, 1 joints
Links:
- link base_link: geometry collision box size=0.255 0.15 0.17; visual box size=0.255 0.15 0.17
Joints:
- joint base_to_laser: origin xyz=0 0 0.15 rpy=0 0 0 -> xyz=0 0 0.02 rpy=0 0 0

Commit message: SLAM + AMCL + EKF stable configuration

File: src/rc_description/urdf/rc_base.urdf (robot description, URDF)
Before this commit: robot rc_car, 2 links, 1 joints
Links:
- link base_link: geometry collision box size=0.255 0.15 0.17; visual box size=0.20 0.15 0.17
